File: lab-supply-control-board.sch (KiCad schematic (older format))
At the start: 69 parts, among them J1 Conn_01x02, J10 AVR-ISP-6, J2 Conn_01x02, J3 Conn_01x02, J4 Conn_01x02, J5 Conn_01x02, J6 Conn_01x05_Male, J7 Conn_01x05_Male, J8 Conn_01x05_Male, J9 USB_B_Micro, Q1 2N3904, Q2 2N3904, Q3 2N3904, U1 MCP4716AxT-ECH, U2 MCP4716AxT-ECH, U3 ATmega328P-AU, U4 LM4040DBZ-2.5, U5 24LC04, U6 LK112M33TR, U7 EA_eDIP320J-8LA, U8 ADuM1200AR, Y1 Crystal_GND24

Commit message: Updated Control Board
Parts:
- removed J3: Conn_01x02, symbol Connector_Generic:Conn_01x02
- removed U7: EA_eDIP320J-8LA, symbol Display_Graphic:EA_eDIP320J-8LA
- removed U8: ADuM1200AR, Package_SO:SOIC-8_3.9x4.9mm_P1.27mm, symbol Isolator:ADuM1200AR
- added J?: 1x04 JST, Connectors_JST:JST_XH_B05B-XH-A_04x2.50mm_Straight, symbol Connector:Conn_01x04_Male
- added J?: 0.1\" Header, Connector_PinHeader_2.54mm:PinHeader_1x11_P2.54mm_Vertical, symbol Connector_Generic:Conn_01x11
- added R?: 100, Resistors_SMD:R_0603_HandSoldering, symbol Device:R_US
- added R? (x3): 10k, Rays Footprints:R_0805_HandSoldering, symbol Device:R_US
- added R? (x3): 19.4k, Rays Footprints:R_0805_HandSoldering, symbol Device:R_US
- added U? (x2): TXS0102DCT, Package_SO:SSOP-8_2.95x2.8mm_P0.65mm, symbol Logic_LevelTranslator:TXS0102DCT
- J4: value Conn_01x02 -> 0.1\" Header
- J8: value Conn_01x05_Male -> 1x04 JST
- J?: renamed from TP3; value Mount Hole -> 0.1\" Header
Connections:
- net labels added: +3.3V, DISP_CS, DISP_CS_3.3, DISP_DC, DISP_DC_3,3, DISP_DC_3.3, MISO_3.3, MOSI_3.3, SCK_3.3, TS_CS, TS_CS_3.3, TS_IRQ, USB_D+, USB_D-
- net labels removed: CS, GNDD, UCB_D-, USB+D+, Vprobe1, Vprobe2, Vprobe3, Vprobe4
- wire segments 259 -> 293
Other:
- note added: "5V <-> 3.3V\nLevel Translator\nReplace with TXS0104 in SOIC-14"
- note added: "Board Level I/O"
- note added: "I/O to Display Board"
- note added: "I2C Circuitry: SDA/SCL LED indicators, pull-ups"
- note added: "I2C Port\n(Expansion)"
- note added: "SPI Port\n(Expansion)"
- note removed: "1"
- note removed: "320x240\nDisplay"
- note removed: "5V <-> 3.3V\nLevel Translator"
- note removed: "I2C Circuitry"
- note removed: "SPI Port"
- moved on the sheet: J10, J4, J6, J8, J9, J?, R1, R2, R4, R5, R6, R7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

Commit message: Added PB0/1 IO Port
Parts:
- added J?: 0.1\" Header, Connector_PinHeader_2.54mm:PinHeader_1x04_P2.54mm_Vertical, symbol Connector_Generic:Conn_01x04
Connections:
- net labels added: PB1_IO, PBO0_IO
- wire segments 293 -> 298
Other:
- moved on the sheet: J8, J?
Changed lines of the file:
@@
 L Connector:Conn_01x04_Male J8
 U 1 1 5EFA5054
-P 9550 8300
-F 0 "J8" H 9800 8650 50  0000 R CNN
-F 1 "1x04 JST" H 10000 8550 50  0000 R CNN
-F 2 "Connectors_JST:JST_XH_B05B-XH-A_04x2.50mm_Straight" H 9550 8300 50  0001 C CNN
-F 3 "B5B-XH-A(LF)(SN)" H 9550 8300 50  0001 C CNN
-	1    9550 8300
+P 9050 8250
+F 0 "J8" H 9300 8600 50  0000 R CNN
+F 1 "1x04 JST" H 9500 8500 50  0000 R CNN
+F 2 "Connectors_JST:JST_XH_B05B-XH-A_04x2.50mm_Straight" H 9050 8250 50  0001 C CNN
+F 3 "B5B-XH-A(LF)(SN)" H 9050 8250 50  0001 C CNN
+	1    9050 8250
 	1    0    0    -1
 $EndComp
@@
 Wire Wire Line
 	3100 2000 3150 2000
-Text GLabel 9800 8500 2    60   Input ~ 0
+Text GLabel 9300 8450 2    60   Input ~ 0
 SCK
-Text GLabel 9800 8400 2    60   Input ~ 0
+Text GLabel 9300 8350 2    60   Input ~ 0
 MISO
-Text GLabel 9800 8300 2    60   Input ~ 0
+Text GLabel 9300 8250 2    60   Input ~ 0
 MOSI
 Wire Wire Line
-	9750 8200 9800 8200
-Wire Wire Line
-	9800 8300 9750 8300
-Wire Wire Line
-	9750 8400 9800 8400
-Wire Wire Line
-	9800 8500 9750 8500
+	9250 8150 9300 8150
+Wire Wire Line
+	9300 8250 9250 8250
+Wire Wire Line
+	9250 8350 9300 8350
+Wire Wire Line
+	9300 8450 9250 8450
 $Comp
 L Connector_Generic:Conn_01x02 J2
@@
 Wire Notes Line
 	11350 550  15350 550
-Text Notes 9550 7800 0    59   ~ 0
+Text Notes 9050 7750 0    59   ~ 0
   SPI Port\n(Expansion)
 Wire Wire Line
@@
 L Connector:Conn_01x04_Male J?
 U 1 1 5F5CB5DA
-P 10450 8300
-F 0 "J?" H 10700 8650 50  0000 R CNN
-F 1 "1x04 JST" H 10900 8550 50  0000 R CNN
-F 2 "Connectors_JST:JST_XH_B05B-XH-A_04x2.50mm_Straight" H 10450 8300 50  0001 C CNN
-F 3 "B5B-XH-A(LF)(SN)" H 10450 8300 50  0001 C CNN
-	1    10450 8300
-	1    0    0    -1
-$EndComp
-Text GLabel 10750 8400 2    50   Input ~ 0
+P 9950 8250
+F 0 "J?" H 10200 8600 50  0000 R CNN
+F 1 "1x04 JST" H 10400 8500 50  0000 R CNN
+F 2 "Connectors_JST:JST_XH_B05B-XH-A_04x2.50mm_Straight" H 9950 8250 50  0001 C CNN
+F 3 "B5B-XH-A(LF)(SN)" H 9950 8250 50  0001 C CNN
+	1    9950 8250
+	1    0    0    -1
+$EndComp
+Text GLabel 10250 8350 2    50   Input ~ 0
 SDA
-Text GLabel 10750 8300 2    50   Input ~ 0
+Text GLabel 10250 8250 2    50   Input ~ 0
 SCL
-Text GLabel 10750 8200 2    50   Input ~ 0
+Text GLabel 10250 8150 2    50   Input ~ 0
 +5V
 $Comp
 L power:GND #PWR?
 U 1 1 5F5DF6E0
-P 10750 8550
-F 0 "#PWR?" H 10750 8300 50  0001 C CNN
-F 1 "GND" H 10755 8377 50  0001 C CNN
-F 2 "" H 10750 8550 50  0001 C CNN
-F 3 "" H 10750 8550 50  0001 C CNN
-	1    10750 8550
-	1    0    0    -1
-$EndComp
-Wire Wire Line
-	10650 8200 10750 8200
-Wire Wire Line
-	10750 8300 10650 8300
-Wire Wire Line
-	10650 8400 10750 8400
-Wire Wire Line
-	10650 8500 10750 8500
-Wire Wire Line
-	10750 8500 10750 8550
+P 10250 8500
+F 0 "#PWR?" H 10250 8250 50  0001 C CNN
+F 1 "GND" H 10255 8327 50  0001 C CNN
+F 2 "" H 10250 8500 50  0001 C CNN
+F 3 "" H 10250 8500 50  0001 C CNN
+	1    10250 8500
+	1    0    0    -1
+$EndComp
+Wire Wire Line
+	10150 8150 10250 8150
+Wire Wire Line
+	10250 8250 10150 8250
+Wire Wire Line
+	10150 8350 10250 8350
+Wire Wire Line
+	10150 8450 10250 8450
+Wire Wire Line
+	10250 8450 10250 8500
 $Comp
 L Connector_Generic:Conn_01x07 J?
@@
 	1    0    0    -1
 $EndComp
-Text Notes 10400 7800 0    59   ~ 0
+Text Notes 9900 7750 0    59   ~ 0
   I2C Port\n(Expansion)
 Text GLabel 8300 7650 0    50   Input ~ 0
@@
 TS_CS
 Wire Wire Line
-	3100 1500 3600 1500
-Wire Wire Line
-	3100 1600 3600 1600
-Wire Wire Line
 	3100 1700 3350 1700
 Wire Wire Line
@@
 Wire Wire Line
 	3350 4600 3450 4600
-Text GLabel 9800 8200 2    50   Input ~ 0
+Text GLabel 9300 8150 2    50   Input ~ 0
 TS_CS
 Wire Wire Line
@@
 Text GLabel 12350 8100 0    50   Input ~ 0
 SCK
+Text GLabel 4000 1500 2    50   Input ~ 0
+PBO0_IO
+Text GLabel 4000 1600 2    50   Input ~ 0
+PB1_IO
+Wire Wire Line
+	3100 1500 4000 1500
+Wire Wire Line
+	3100 1600 4000 1600
+Text GLabel 11200 8250 2    50   Input ~ 0
+PBO0_IO
+Text GLabel 11200 8350 2    50   Input ~ 0
+PB1_IO
+$Comp
+L Connector_Generic:Conn_01x04 J?
+U 1 1 5EDC6A75
+P 10900 8250
+F 0 "J?" H 10750 7500 50  0000 L CNN
+F 1 "0.1\" Header" H 10550 7400 50  0000 L CNN
+F 2 "Connector_PinHeader_2.54mm:PinHeader_1x04_P2.54mm_Vertical" H 11100 8250 50  0001 C CNN
+F 3 "" H 11100 8250 50  0001 C CNN
+	1    10900 8250
+	-1   0    0    -1
+$EndComp
+Wire Wire Line
+	11200 8250 11100 8250
+$Comp
+L power:GND #PWR?
+U 1 1 5EE30B57
+P 11150 8500
+F 0 "#PWR?" H 11150 8250 50  0001 C CNN
+F 1 "GND" H 11155 8327 50  0001 C CNN
+F 2 "" H 11150 8500 50  0001 C CNN
+F 3 "" H 11150 8500 50  0001 C CNN
+	1    11150 8500
+	1    0    0    -1
+$EndComp
+Wire Wire Line
+	11150 8500 11150 8450
+Wire Wire Line
+	11150 8450 11100 8450
+Wire Wire Line
+	11100 8350 11200 8350
+Text GLabel 11200 8150 2    50   Input ~ 0
++5V
+Wire Wire Line
+	11200 8150 11100 8150
 $EndSCHEMATC

Commit message: Added FT232
Parts:
- added U?: FT232RL, Package_SO:SSOP-28_5.3x10.2mm_P0.65mm, symbol Interface_USB:FT232RL
Other:
- note added: "Do we want one of these?"
- moved on the sheet: R?

Commit message: Worked over the schematic, started layout
Parts:
- removed C5: 1u, Capacitors_SMD:C_0603_HandSoldering, symbol Device:C
- removed C6: 10u, Capacitors_SMD:CP_Elec_4x4.5, symbol Device:CP1
- removed J2: Conn_01x02, symbol Connector_Generic:Conn_01x02
- removed R11: 1K, Resistors_SMD:R_0805_HandSoldering, symbol Device:R
- removed R19, R24, R25, R26: 10k, Resistors_SMD:R_0805_HandSoldering, symbol Device:R
- removed R2, R4, R6, R7, R8, R9: 0.1, Rays Footprints:R_0805_HandSoldering, symbol Device:R_US
- removed R20, R21: 2k, Resistors_SMD:R_0805_HandSoldering, symbol Device:R
- removed R?: 10k, Rays Footprints:R_0805_HandSoldering, symbol Device:R_US
- removed R?: 19.4k, Rays Footprints:R_0805_HandSoldering, symbol Device:R_US
- removed U6: LK112M33TR, Package_TO_SOT_SMD:SOT-23-5, symbol Regulator_Linear:LK112M33TR
- removed U? (x2): TXS0102DCT, Package_SO:SSOP-8_2.95x2.8mm_P0.65mm, symbol Logic_LevelTranslator:TXS0102DCT
- added C10, C9: 1.0u, Rays Footprints:C_0805_HandSoldering, symbol Device:C_Small
- added C13, C7, C8: 0.1u, Rays Footprints:C_0805_HandSoldering, symbol Device:C
- added D3, D4, D6: LED, LED_SMD:LED_0805_2012Metric_Pad1.15x1.40mm_HandSolder, symbol Device:LED
- added J8, J9: 0.1\" Header, Connector_PinHeader_2.54mm:PinHeader_1x02_P2.54mm_Vertical, symbol Connector_Generic:Conn_01x02
- added Q1, Q2, Q6, Q7: BSS138, Package_TO_SOT_SMD:SOT-23, symbol Transistor_FET:BSS138
- added R11, R12, R13, R14, R23, R24, R25, R26, R27, R34, R35, R36, R37, R41, R42, R43, R44: 10k, Rays Footprints:R_0805_HandSoldering, symbol Device:R_US
- added R16, R28, R29: 50k, Rays Footprints:R_0805_HandSoldering, symbol Device:R_US
- added R17, R19, R45, R46: 2k, Rays Footprints:R_0805_HandSoldering, symbol Device:R_US
- added R18, R30: 10k/DNP, Rays Footprints:R_0805_HandSoldering, symbol Device:R_US
- added R22, R31: 19.4k/DNP, Rays Footprints:R_0805_HandSoldering, symbol Device:R_US
- added R40: 0, Rays Footprints:R_0805_HandSoldering, symbol Device:R_US
- added R48: 1.3k, Rays Footprints:R_0805_HandSoldering, symbol Device:R_US
- added U6: MIC5365-3.3YD5, Package_TO_SOT_SMD:SOT-23-5, symbol Regulator_Linear:MIC5365-3.3YD5
- C1: renamed from C4; footprint Capacitors_SMD:C_0805_HandSoldering -> Rays Footprints:C_0805_HandSoldering
- C11: renamed from C2; footprint Capacitors_SMD:CP_Elec_4x4.5 -> Capacitor_SMD:CP_Elec_4x4.5
- C12: renamed from C3; value 100n -> 0.1u; footprint Capacitors_SMD:C_0805_HandSoldering -> Rays Footprints:C_0805_HandSoldering
- C2: renamed from C7; footprint Capacitors_SMD:C_0805_HandSoldering -> Rays Footprints:C_0805_HandSoldering
- C3: renamed from C8; value 100n -> 15p; footprint Capacitors_SMD:C_0603_HandSoldering -> Rays Footprints:C_0603_HandSoldering
- C4: renamed from C1; footprint Rays Footprints:C_0603_HandSoldering -> Rays Footprints:C_0805_HandSoldering
- C5: renamed from C9; value 100n -> 15p; footprint Capacitors_SMD:C_0603_HandSoldering -> Rays Footprints:C_0603_HandSoldering
- C6: renamed from C10; footprint Rays Footprints:C_0603_HandSoldering -> Rays Footprints:C_0805_HandSoldering
- D1: renamed from D2; footprint LEDs:LED_0805_HandSoldering -> LED_SMD:LED_0805_2012Metric_Pad1.15x1.40mm_HandSolder
- D2: renamed from D3; footprint LEDs:LED_0805_HandSoldering -> LED_SMD:LED_0805_2012Metric_Pad1.15x1.40mm_HandSolder
- D5: renamed from D1; footprint LEDs:LED_0805_HandSoldering -> LED_SMD:LED_0805_2012Metric_Pad1.15x1.40mm_HandSolder
- J1: renamed from J5; value Conn_01x02 -> 0.1\" header; footprint (none) -> Connector_PinHeader_2.54mm:PinHeader_1x02_P2.54mm_Vertical
- J10: renamed from J9; footprint (none) -> Connector_USB:USB_Micro-B_Molex-105133-0001
- J11: renamed from J?; footprint Connector_PinHeader_2.54mm:PinHeader_1x04_P2.54mm_Vertical -> Connector_PinHeader_2.54mm:PinHeader_1x03_P2.54mm_Vertical; symbol Connector_Generic:Conn_01x04 -> Connector_Generic:Conn_01x03
- J12: renamed from J8; footprint Connectors_JST:JST_XH_B05B-XH-A_04x2.50mm_Straight -> Connector_JST:JST_XH_B4B-XH-A_1x04_P2.50mm_Vertical
- J13: renamed from J?; footprint Connectors_JST:JST_XH_B05B-XH-A_04x2.50mm_Straight -> Connector_JST:JST_XH_B4B-XH-A_1x04_P2.50mm_Vertical
- J14: renamed from J4; footprint (none) -> Connector_PinHeader_2.54mm:PinHeader_1x05_P2.54mm_Vertical; symbol Connector_Generic:Conn_01x04 -> Connector_Generic:Conn_01x05
- J5: renamed from J?; footprint Connector_PinHeader_2.54mm:PinHeader_1x11_P2.54mm_Vertical -> Connector_PinHeader_2.54mm:PinHeader_1x09_P2.54mm_Vertical; symbol Connector_Generic:Conn_01x11 -> Connector_Generic:Conn_01x09
- J6: renamed from J10; footprint (none) -> Rays Footprints:AVR-ISP-6-TH
- J7: renamed from J1; value Conn_01x02 -> 0.1\" Header; footprint (none) -> Connector_PinHeader_2.54mm:PinHeader_1x02_P2.54mm_Vertical
- R1: value 0.1 -> 0/DNP
- R10: renamed from R18; footprint Resistors_SMD:R_0603_HandSoldering -> Rays Footprints:R_0805_HandSoldering
- R15: renamed from R?; footprint Resistors_SMD:R_0603_HandSoldering -> Rays Footprints:R_0805_HandSoldering
- R2: renamed from R12; footprint Resistors_SMD:R_0603_HandSoldering -> Rays Footprints:R_0805_HandSoldering
- R20: renamed from R22; value 4.7k -> 10k; footprint Resistors_SMD:R_0603_HandSoldering -> Rays Footprints:R_0805_HandSoldering
- R21: renamed from R23; value 4.7k -> 10k; footprint Resistors_SMD:R_0603_HandSoldering -> Rays Footprints:R_0805_HandSoldering
- R3: renamed from R13; footprint Resistors_SMD:R_0603_HandSoldering -> Rays Footprints:R_0805_HandSoldering
- R4: renamed from R14; footprint Resistors_SMD:R_0603_HandSoldering -> Rays Footprints:R_0805_HandSoldering
- R47: renamed from R3; value 2K -> 3k; footprint Resistors_SMD:R_0805_HandSoldering -> Rays Footprints:R_0805_HandSoldering
- R5: value 0.1 -> 1k
- R6: renamed from R15; footprint Resistors_SMD:R_0603_HandSoldering -> Rays Footprints:R_0805_HandSoldering
- R8: renamed from R16; footprint Resistors_SMD:R_0603_HandSoldering -> Rays Footprints:R_0805_HandSoldering
- R9: renamed from R17; footprint Resistors_SMD:R_0603_HandSoldering -> Rays Footprints:R_0805_HandSoldering
- TP1: value Mount Hole -> 0.1\" Header
- TP2: footprint Measurement_Points:Test_Point_Keystone_5000-5004_Miniature -> Connector_PinHeader_2.54mm:PinHeader_1x01_P2.54mm_Vertical
- U3: renamed from U5; footprint Housings_SOIC:SOIC-8_3.9x4.9mm_Pitch1.27mm -> Package_SO:SOIC-8_3.9x4.9mm_P1.27mm
- gave numbers to parts that had none: 6
- renumbered J6 to J2, J7 to J3, Q1 to Q3, Q2 to Q4, Q3 to Q5, R10 to R7, U3 to U2, U2 to U5
Connections:
- net labels added: 3.3V, DISP_RESET, DISP_RESET_3.3, LED_PWM, PB2_IO
- net labels removed: DISP_DC_3,3, PB1_IO, PBO0_IO, TS_CS_3.3, TS_IRQ
- wire segments 298 -> 422
Other:
- note added: "- Check for nearby Vcc bypass -"
- note added: "3.3V for Display I/O (remove?)\n- Optional - Use FT232 3V3OUT?"
- note added: "Alternate to using GPIO Pin to reset display"
- note added: "DAC Circuitry: Want Vout up to 5V (Vdd=5V)"
- note added: "For Debug"
- note added: "I2C Circuitry: SDA/SCL LED indicators, I2C pull-ups (ATMEGA328P=20k)"
- note added: "Level shifters\n- Use only resistor divider for uni-directional\n- Use FET/pull-ups for bi-directional (not needed - delete?)"
- note added: "MCP4716: Only acts as slave\nVih = 0.7xVdd -> requires 5V signaling from CPU\nVoh = 0.3xVdd\nVref = 2.5V, configure DAC gain = 2\n- Prevents VOUT_DAC from exceeding 5.0V\n- Cleans up noise from supply. If Vref=Vdd, PSRR ~~0dB"
- note added: "Main Bypass"
- note added: "PWM Output\n(if DISP_RESET unused)"
- note added: "Power Indicators (1mA/5mW ea)"
- note added: "Power Supply"
- note added: "\nWrite\nProtect"
- note removed: "3.3V for Display"
- note removed: "5V <-> 3.3V\nLevel Translator\nReplace with TXS0104 in SOIC-14"
- note removed: "DAC Circuitry"
- note removed: "Do we want one of these?"
- note removed: "I2C Circuitry: SDA/SCL LED indicators, pull-ups"
- moved on the sheet: C1, C11, C12, C2, C3, C4, C5, C6, D1, D2, D5, J1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

Commit message: schematic tweak
Other:
- note added: "EEPROM\n- Not clear this is at all needed\n- Remove?"
- note added: "MCP4716: Only acts as slave\nVih = 0.7xVdd -> requires 5V signaling from CPU\nVoh = 0.3xVdd\nVref = 2.5V, configure DAC gain = 2\n- Prevents VOUT_DAC from exceeding 5.0V\n- Cleans up noise from supply. If Vref=Vdd, PSRR ~~0dB\n- Could consider a buffer. Want Rload ~~2k"
- note removed: "EEPROM"
- note removed: "MCP4716: Only acts as slave\nVih = 0.7xVdd -> requires 5V signaling from CPU\nVoh = 0.3xVdd\nVref = 2.5V, configure DAC gain = 2\n- Prevents VOUT_DAC from exceeding 5.0V\n- Cleans up noise from supply. If Vref=Vdd, PSRR ~~0dB"
- moved on the sheet: C4, C6, R7, TP1, U1, U4, U5

Commit message: Updates to schematic, started control board layout
Parts:
- removed C10, C9: 1.0u, Rays Footprints:C_0805_HandSoldering, symbol Device:C_Small
- removed Q1, Q2, Q6: BSS138, Package_TO_SOT_SMD:SOT-23, symbol Transistor_FET:BSS138
- removed R11, R12, R13, R14, R34, R35: 10k, Rays Footprints:R_0805_HandSoldering, symbol Device:R_US
- removed U6: MIC5365-3.3YD5, Package_TO_SOT_SMD:SOT-23-5, symbol Regulator_Linear:MIC5365-3.3YD5
- added C14: 0.1u, Rays Footprints:C_0805_HandSoldering, symbol Device:C_Small
- added MTH5: Mount Hole, Rays Footprints:Mount-Hole-#6, symbol Connector_Generic:Conn_01x01
- added R49: 1k, Rays Footprints:R_0805_HandSoldering, symbol Device:R_US
- added U8: MCP6002-xSN, Package_SO:SOP-8_3.9x4.9mm_P1.27mm, symbol Amplifier_Operational:MCP6002-xSN
- J2, J3: value Conn_01x05_Male -> JST; footprint Connectors_JST:JST_XH_B05B-XH-A_05x2.50mm_Straight -> Connector_JST:JST_XH_B5B-XH-A_1x05_P2.50mm_Vertical
- R24, R26, R41: value 10k -> 19.4k
- R40: value 0 -> 1k
Connections:
- net labels added: RXD, TXD
- net labels removed: +5VD, 3.3V
- wire segments 422 -> 392
Other:
- note added: "Encoder_1"
- note added: "Encoder_2"
- note added: "Level shifters\n- Resistor dividers provide uni-directional translation\n- FETs provide bi-directional (test circuit)"
- note added: "MCP4716: Only acts as slave\nVih = 0.7xVdd -> requires 5V signaling from CPU\nVref = 2.5V, configure DAC gain = 2\n- Prevents VOUT_DAC from exceeding 5.0V\n- Cleans up noise from supply. If Vref=Vdd, PSRR ~~0dB\n- R/R buffer due to high DAC output impedance"
- note removed: "3.3V for Display I/O (remove?)\n- Optional - Use FT232 3V3OUT?"
- note removed: "Encoder_Other"
- note removed: "Encoder_Vout"
- note removed: "Level shifters\n- Use only resistor divider for uni-directional\n- Use FET/pull-ups for bi-directional (not needed - delete?)"
- note removed: "MCP4716: Only acts as slave\nVih = 0.7xVdd -> requires 5V signaling from CPU\nVoh = 0.3xVdd\nVref = 2.5V, configure DAC gain = 2\n- Prevents VOUT_DAC from exceeding 5.0V\n- Cleans up noise from supply. If Vref=Vdd, PSRR ~~0dB\n- Could consider a buffer. Want Rload ~~2k"
- moved on the sheet: C11, C12, C4, C6, D5, D6, J10, J2, J3, J7, J8, J9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

Commit message: Updated control sch, first full cut at layout
Parts:
- removed C12: 0.1u, Rays Footprints:C_0805_HandSoldering, symbol Device:C
- removed J1: 0.1\" header, Connector_PinHeader_2.54mm:PinHeader_1x02_P2.54mm_Vertical, symbol Connector_Generic:Conn_01x02
- removed R10, R2, R3, R4, R6, R8, R9: 10k, Rays Footprints:R_0805_HandSoldering, symbol Device:R_US
- removed U3: 24LC04, Package_SO:SOIC-8_3.9x4.9mm_P1.27mm, symbol memory:24LC04
- added J1: JST, Connector_JST:JST_XH_B2B-XH-A_1x02_P2.50mm_Vertical, symbol Connector:Conn_01x02_Male
- J14: footprint Connector_PinHeader_2.54mm:PinHeader_1x05_P2.54mm_Vertical -> Connector_PinHeader_2.54mm:PinHeader_1x04_P2.54mm_Vertical; symbol Connector_Generic:Conn_01x05 -> Connector_Generic:Conn_01x04
Connections:
- net labels added: BB_VOUT, BUTTON
- net labels removed: ADC3, VOUT
- wire segments 392 -> 361
Other:
- note added: "Bidirectional"
- note added: "DAC Circuitry: Analog (or digital) Vout up to 5V"
- note added: "FT232 for USB\nProgramming and\nData to PC"
- note added: "I/O to Analog Board\n- BB_VOUT: Output voltage\n- BB_IOUT: Output current\n- BB_ALERT: Error condition"
- note added: "ISP Programming Port\n For Bootloader"
- note added: "Level shifters\n- Resistor dividers provide uni-directional translation\n- FET provides bi-directional (test circuit)"
- note added: "Unidirectional"
- note removed: "- Check for nearby Vcc bypass -"
- note removed: "DAC Circuitry: Want Vout up to 5V (Vdd=5V)"
- note removed: "EEPROM\n- Not clear this is at all needed\n- Remove?"
- note removed: "I/O to Analog Board"
- note removed: "Level shifters\n- Resistor dividers provide uni-directional translation\n- FETs provide bi-directional (test circuit)"
- note removed: "Programming Port"
- note removed: "\nWrite\nProtect"
- moved on the sheet: C14, C4, C6, J4, J5, R15, R18, R22, R30, R31, R7, TP1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

Commit message: Worked on board layouts
Parts:
- removed J10: USB_B_Micro, Connector_USB:USB_Micro-B_Molex-105133-0001, symbol conn:USB_B_Micro
- added J10: USB-Micro, Rays Footprints:USB-Micro-AMPHENOL_10118194-0001LF, symbol Rays_Symbols:USB-Micro-AMPHENOL_10118194-0001LF
- J1: footprint Connector_JST:JST_XH_B2B-XH-A_1x02_P2.50mm_Vertical -> Connector_JST:JST_XH_B4B-XH-A_1x04_P2.50mm_Vertical; symbol Connector:Conn_01x02_Male -> Connector:Conn_01x04_Male
- J14: footprint Connector_PinHeader_2.54mm:PinHeader_1x04_P2.54mm_Vertical -> Connector_JST:JST_XH_B5B-XH-A_1x05_P2.50mm_Vertical; symbol Connector_Generic:Conn_01x04 -> Connector_Generic:Conn_01x05
- J4: footprint Connector_PinHeader_2.54mm:PinHeader_1x07_P2.54mm_Vertical -> Connector_JST:JST_XH_B5B-XH-A_1x05_P2.50mm_Vertical; symbol Connector_Generic:Conn_01x07 -> Connector_Generic:Conn_01x05
- J5: footprint Connector_PinHeader_2.54mm:PinHeader_1x09_P2.54mm_Vertical -> Connector_JST:JST_XH_B9B-XH-A_1x09_P2.50mm_Vertical
- TP1: footprint Connector_PinHeader_2.54mm:PinHeader_1x04_P2.54mm_Vertical -> Connector_JST:JST_XH_B4B-XH-A_1x04_P2.50mm_Vertical
- U1: value MCP4716AxT-ECH -> MCP4716A0T-ECH
- U5: value MCP4716AxT-ECH -> MCP4716A1T-ECH
Connections:
- net +5V: now also J1.4 (Pin_4), J3.5 (Pin_5), J5.9 (Pin_9), J10.1; no longer J3.1 (Pin_1), J5.1 (Pin_1)
- net ADC0: now also J14.4 (Pin_4), U2.22 (ADC7); no longer J14.2 (Pin_2), U2.23 (PC0)
- net ADC1: now also U2.23 (PC0); no longer U2.24 (PC1)
- net ADC2: now also J14.2 (Pin_2), U2.24 (PC1); no longer J14.4 (Pin_4), U2.25 (PC2)
- net BB_ALERT: now also J4.2 (Pin_2); no longer J4.4 (Pin_4)
- net DISP_CS_3.3: now also J5.8 (Pin_8); no longer J5.2 (Pin_2)
- net DISP_DC_3.3: now also J5.7 (Pin_7); no longer J5.3 (Pin_3)
- net DISP_RESET_3.3: now also J5.2 (Pin_2); no longer J5.8 (Pin_8)
- net GND: now also J14.5 (Pin_5), J3.1 (Pin_1), J4.5 (Pin_5), J5.1 (Pin_1), J10.5, J10.S1 (SHIELD), J10.S2 (SHIELD), J10.S3 (SHIELD), J10.S4 (SHIELD), J10.S5 (SHIELD), J10.S6 (SHIELD); no longer J14.1 (Pin_1), J3.5 (Pin_5), J4.7 (Pin_7), J5.9 (Pin_9)
- net MISO_3.3: now also J5.6 (Pin_6); no longer J5.4 (Pin_4)
- net SCK_3.3: now also J5.4 (Pin_4); no longer J5.6 (Pin_6)
- net SCL: now also J4.3 (Pin_3); no longer J4.5 (Pin_5)
- net SDA: now also J4.4 (Pin_4); no longer J4.6 (Pin_6)
- net USB_D+: now also J10.3
- net USB_D-: now also J10.2
- net at R15.2, R18.2, R22.2: now also J5.3 (Pin_3); no longer J5.7 (Pin_7)
- net RxLED: now reaches D3.1 (K), R45.1
- net TxLED: now reaches D4.1 (K), R46.1
- net BB_IOUT renamed ADC3
- net ADC3: now also J14.1 (Pin_1); no longer J4.3 (Pin_3)
- removed net BB_VOUT: J4.2 (Pin_2), U2.22 (ADC7)
- net BUTTON renamed BUTTON2
- new net BUTTON1: J1.3 (Pin_3), U2.25 (PC2)
Other:
- note added: "Buttons"
- note added: "I2C:0x60"
- note added: "I2C:0x61"
- note added: "Main Bypass\n10uF Max"
- note removed: "Main Bypass"
- moved on the sheet: D3, D4, J7, J8, J9
