File: lab-supply-control-board.sch (KiCad schematic (older format))
At the start: 88 parts, among them J1 JST, J10 USB-Micro, J11 0.1\" Header, J12 1x05 JST, J13 1x04 JST, J14 0.1\" Header, J15 0.1\" Header, J2 JST, J3 JST, J4 0.1\" Header, J5 0.1\" Header, J6 AVR-ISP-6, J7 0.1\" Header, J8 0.1\" Header, J9 0.1\" Header, Q3 2N3904, Q4 2N3904, Q5 2N3904, Q7 BSS138, U1 MCP4716A0T-ECH, U2 ATmega328P-AU, U4 LM4040DBZ-2.5, U5 MCP4716A1T-ECH, U7 FT232RL, U8 MCP6002-xSN, Y1 Crystal_GND24

Commit message: finalized before PCB orders
Parts:
- removed Q7: BSS138, Package_TO_SOT_SMD:SOT-23, symbol Transistor_FET:BSS138
- removed R36, R37: 10k, Rays Footprints:R_0805_HandSoldering, symbol Device:R_US
Connections:
- net labels removed: TS_CS
- wire segments 370 -> 357
Other:
- note added: "Alternate to using\nGPIO Pin to reset display"
- note added: "Level shifters\n- Resistor dividers provide uni-directional translation"
- note removed: "Alternate to using GPIO Pin to reset display"
- note removed: "Bidirectional (for testing)"
- note removed: "Level shifters\n- Resistor dividers provide uni-directional translation\n- FET provides bi-directional (test circuit)"
- note removed: "Unidirectional"
- moved on the sheet: J4, J5, J6, R15, R18, R22, R24, R25, R26, R27, R30, R31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
