File: lab-supply.sch (KiCad schematic (older format))
At the start: 40 parts, among them Q1 Q_NPN_BCE, U1 AD8208, U2 MAX1719EUT, U3 MP8862GQ, U4 MCP4716AxT-ECH, U5 LM4040DBZ-2.5, U6 MCP4716AxT-ECH

Commit message: Kept working on the design
Parts:
- removed C7: 10u, Capacitor_SMD:CP_Elec_4x4.5, symbol Device:CP1_Small
- removed R5: 25k, Rays Footprints:R_0805_HandSoldering, symbol Device:R_US
- removed TP4: Mount Hole, Connector_PinHeader_2.54mm:PinHeader_1x04_P2.54mm_Vertical, symbol Connector_Generic:Conn_01x04
- removed U4, U6: MCP4716AxT-ECH, Package_TO_SOT_SMD:SOT-23-6_Handsoldering, symbol Rays_Symbols:MCP4716AxT-ECH
- removed U5: LM4040DBZ-2.5, Package_TO_SOT_SMD:SOT-23, symbol Reference_Voltage:LM4040DBZ-2.5
- added C10, C11, C8: 22u, Rays Footprints:C_1210_HandSoldering, symbol Device:C_Small
- added C16: 0.1u, Rays Footprints:C_0603_HandSoldering, symbol Device:C_Small
- added R6: 300k, Rays Footprints:R_0805_HandSoldering, symbol Device:R_US
- added R8: 0, Rays Footprints:R_0805_HandSoldering, symbol Device:R_US
- C12, C13: value 0.1u -> 22u; footprint Rays Footprints:C_0603_HandSoldering -> Rays Footprints:C_1210_HandSoldering
- TP1: value Mount Hole -> Input Power
- TP2: value Mount Hole -> Output Power
- TP3: footprint Connector_PinHeader_2.54mm:PinHeader_1x11_P2.54mm_Vertical -> Connector_PinHeader_2.54mm:PinHeader_1x07_P2.54mm_Vertical; symbol Connector_Generic:Conn_01x11 -> Connector_Generic:Conn_01x07
- gave numbers to parts that had none: 1
- renumbered C5 to C1, C11 to C14, C16 to C15, C15 to C17, C2 to C18, C3 to C19, C6 to C2, C1 to C3, C9 to C5, C10 to C6, C8 to C7, C14 to C9, R2 to R1, R3 to R2, R1 to R3, R11 to R5, R6 to R9, U3 to U1, U1 to U2, U2 to U3
Connections:
- net labels added: BB_ALERT, SCL, SDA
- net labels removed: BB_ALT, BB_SCL, BB_SDA, DAC1_SCL, DAC1_SDA, DAC2_SCL, DAC2_SDA, VOUT_DAC1, VOUT_DAC2, VREF_2.5
- wire segments 174 -> 153
Other:
- note added: "<----\n5mA min load"
- note added: "Gain = 20V/V\nBB_IOUT = Iout x 3.0\n1.5A = 4.5V"
- note removed: "---->\n5mA min load"
- note removed: "Gain = 20V/V\nBB_IOUT = Iout x 2.0"
- moved on the sheet: C1, C14, C15, C17, C18, C19, C2, C3, C4, C5, C6, C7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

Commit message: Updated control sch, first full cut at layout
Parts:
- removed R6: 300k, Rays Footprints:R_0805_HandSoldering, symbol Device:R_US
- added U?: INA181, Package_TO_SOT_SMD:SOT-23-6_Handsoldering, symbol Amplifier_Current:INA181
Connections:
- wire segments 153 -> 154
Other:
- note added: "Gain = 20V/V\nBB_IOUT = Iout x 2.0\n1.5A = 3.0V"
- note removed: "Gain = 20V/V\nBB_IOUT = Iout x 3.0\n1.5A = 4.5V"
- moved on the sheet: C9
Changed lines of the file:
@@
 	0    1    1    0
 $EndComp
-Text GLabel 7050 1700 2    50   Input ~ 0
+Text GLabel 6650 1500 2    50   Input ~ 0
 BB_IOUT
 Text Notes 5600 4100 0    79   ~ 0
@@
 Wire Wire Line
 	7350 5200 7350 5150
-Text GLabel 5850 1500 0    50   Input ~ 0
+Text GLabel 5950 1850 0    50   Input ~ 0
 +5V
-$Comp
-L power:GND #PWR0115
-U 1 1 5EEECEBC
-P 6550 1250
-F 0 "#PWR0115" H 6550 1000 50  0001 C CNN
-F 1 "GND" H 6555 1077 50  0001 C CNN
-F 2 "" H 6550 1250 50  0001 C CNN
-F 3 "" H 6550 1250 50  0001 C CNN
-	1    6550 1250
-	-1   0    0    1
-$EndComp
 $Comp
 L Amplifier_Current:AD8208 U2
 U 1 1 5EEF2A9E
-P 6550 1700
-F 0 "U2" H 6700 1200 50  0000 C CNN
-F 1 "AD8208" H 6800 1300 50  0000 C CNN
-F 2 "Package_SO:SOIC-8_3.9x4.9mm_P1.27mm" H 6600 1350 50  0001 L CNN
-F 3 "https://www.analog.com/media/en/technical-documentation/data-sheets/AD8208.pdf" H 7200 1000 50  0001 C CNN
-	1    6550 1700
+P 8050 400
+F 0 "U2" H 8200 -100 50  0000 C CNN
+F 1 "AD8208" H 8300 0   50  0000 C CNN
+F 2 "Package_SO:SOIC-8_3.9x4.9mm_P1.27mm" H 8100 50  50  0001 L CNN
+F 3 "https://www.analog.com/media/en/technical-documentation/data-sheets/AD8208.pdf" H 8700 -300 50  0001 C CNN
+	1    8050 400
 	1    0    0    1
 $EndComp
-Wire Wire Line
-	6550 1250 6550 1300
-Wire Wire Line
-	7050 1700 7000 1700
 Text Notes 7100 1450 0    79   ~ 0
-Gain = 20V/V\nBB_IOUT = Iout x 3.0\n1.5A = 4.5V
-Wire Wire Line
-	6150 1600 6100 1600
-Wire Wire Line
-	6100 1600 6100 1700
-Wire Wire Line
-	6100 1700 6150 1700
+Gain = 20V/V\nBB_IOUT = Iout x 2.0\n1.5A = 3.0V
 $Comp
 L Rays_Symbols:MP8862GQ U1
@@
 	2550 5200 2450 5200
 Wire Wire Line
-	5950 1850 5950 1900
+	6100 2200 6100 2250
 $Comp
 L power:GND #PWR0105
 U 1 1 5F4919A4
-P 5950 1900
-F 0 "#PWR0105" H 5950 1650 50  0001 C CNN
-F 1 "GND" H 5955 1727 50  0001 C CNN
-F 2 "" H 5950 1900 50  0001 C CNN
-F 3 "" H 5950 1900 50  0001 C CNN
-	1    5950 1900
+P 6100 2250
+F 0 "#PWR0105" H 6100 2000 50  0001 C CNN
+F 1 "GND" H 6105 2077 50  0001 C CNN
+F 2 "" H 6100 2250 50  0001 C CNN
+F 3 "" H 6100 2250 50  0001 C CNN
+	1    6100 2250
 	1    0    0    -1
 $EndComp
@@
 L Device:C_Small C9
 U 1 1 5F4919AF
-P 5950 1750
-F 0 "C9" H 6150 1700 50  0000 C CNN
-F 1 "0.1u" H 6150 1800 50  0000 C CNN
-F 2 "Rays Footprints:C_0603_HandSoldering" H 5950 1750 50  0001 C CNN
-F 3 "~" H 5950 1750 50  0001 C CNN
-	1    5950 1750
-	-1   0    0    1
-$EndComp
-Wire Wire Line
-	5850 1500 5950 1500
-Wire Wire Line
-	5950 1500 5950 1650
-Connection ~ 5950 1500
-Wire Wire Line
-	5950 1500 6150 1500
+P 6100 2100
+F 0 "C9" H 6300 2050 50  0000 C CNN
+F 1 "0.1u" H 6300 2150 50  0000 C CNN
+F 2 "Rays Footprints:C_0603_HandSoldering" H 6100 2100 50  0001 C CNN
+F 3 "~" H 6100 2100 50  0001 C CNN
+	1    6100 2100
+	-1   0    0    1
+$EndComp
+Wire Wire Line
+	6100 1850 6100 2000
 Text GLabel 2450 4900 0    50   Input ~ 0
 BB_IOUT
@@
 Connection ~ 5900 2500
 Wire Wire Line
-	6350 2100 6350 2500
-Wire Wire Line
-	6750 2100 6750 2500
-Wire Wire Line
 	5900 2500 6350 2500
 Connection ~ 6350 2500
@@
 Wire Wire Line
 	8100 2200 8100 2250
-$Comp
-L Device:R_US R6
-U 1 1 5EDB07AF
-P 6550 1000
-F 0 "R6" V 6500 800 50  0000 C CNN
-F 1 "300k" V 6500 1150 50  0000 C CNN
-F 2 "Rays Footprints:R_0805_HandSoldering" V 6590 990 50  0001 C CNN
-F 3 "https://www.digikey.com/product-detail/en/bourns-inc/CRL2512-JW-R100ELF/CRL2512-JW-R100ELFCT-ND/5775016" H 6550 1000 50  0001 C CNN
-	1    6550 1000
-	0    1    1    0
-$EndComp
-Wire Wire Line
-	6400 1000 6100 1000
-Wire Wire Line
-	6100 1000 6100 1600
-Connection ~ 6100 1600
-Wire Wire Line
-	6700 1000 7000 1000
-Wire Wire Line
-	7000 1000 7000 1700
-Connection ~ 7000 1700
-Wire Wire Line
-	7000 1700 6950 1700
 Text Notes 8700 4100 1    79   ~ 0
 <----\n5mA min load
@@
 	-1   0    0    -1
 $EndComp
+$Comp
+L Amplifier_Current:INA181 U?
+U 1 1 5ED63FC9
+P 6550 2050
+F 0 "U?" V 6900 1900 50  0000 C CNN
+F 1 "INA181" V 6800 1850 50  0000 C CNN
+F 2 "Package_TO_SOT_SMD:SOT-23-6_Handsoldering" H 6600 2100 50  0001 C CNN
+F 3 "https://www.digikey.com/product-detail/en/texas-instruments/INA181A1IDBVR/296-47656-1-ND/8133025" H 6700 2200 50  0001 C CNN
+	1    6550 2050
+	0    -1   -1   0
+$EndComp
+$Comp
+L power:GND #PWR?
+U 1 1 5ED64732
+P 6900 2200
+F 0 "#PWR?" H 6900 1950 50  0001 C CNN
+F 1 "GND" H 6905 2027 50  0001 C CNN
+F 2 "" H 6900 2200 50  0001 C CNN
+F 3 "" H 6900 2200 50  0001 C CNN
+	1    6900 2200
+	1    0    0    -1
+$EndComp
+Wire Wire Line
+	5950 1850 6100 1850
+Wire Wire Line
+	6900 2200 6900 2150
+$Comp
+L power:GND #PWR?
+U 1 1 5EDA5247
+P 6900 2000
+F 0 "#PWR?" H 6900 1750 50  0001 C CNN
+F 1 "GND" H 6905 1827 50  0001 C CNN
+F 2 "" H 6900 2000 50  0001 C CNN
+F 3 "" H 6900 2000 50  0001 C CNN
+	1    6900 2000
+	1    0    0    -1
+$EndComp
+Wire Wire Line
+	6900 2000 6900 1950
+Wire Wire Line
+	6900 1950 6850 1950
+Wire Wire Line
+	6900 2150 6850 2150
+Wire Wire Line
+	6450 2350 6450 2400
+Wire Wire Line
+	6450 2400 6350 2400
+Wire Wire Line
+	6350 2400 6350 2500
+Wire Wire Line
+	6650 2350 6650 2400
+Wire Wire Line
+	6650 2400 6750 2400
+Wire Wire Line
+	6750 2400 6750 2500
+Wire Wire Line
+	6100 1850 6250 1850
+Wire Wire Line
+	6250 1850 6250 2150
+Connection ~ 6100 1850
+Wire Wire Line
+	6550 1500 6650 1500
+Wire Wire Line
+	6550 1500 6550 1750
 $EndSCHEMATC

Commit message: Worked on board layouts
Parts:
- removed U2: AD8208, Package_SO:SOIC-8_3.9x4.9mm_P1.27mm, symbol Amplifier_Current:AD8208
- removed U?: INA181, Package_TO_SOT_SMD:SOT-23-6_Handsoldering, symbol Amplifier_Current:INA181
- added JP1, JP2: Jumper, Rays Footprints:SolderJumper_3_Pad, symbol Jumper:SolderJumper_3_Open
- added R?: DNP, Rays Footprints:R_0805_HandSoldering, symbol Device:R_US
- added U2: INA220, Package_SO:VSSOP-10_3x3mm_P0.5mm, symbol Analog_ADC:INA226
- TP3: footprint Connector_PinHeader_2.54mm:PinHeader_1x07_P2.54mm_Vertical -> Connector_PinHeader_2.54mm:PinHeader_1x05_P2.54mm_Vertical; symbol Connector_Generic:Conn_01x07 -> Connector_Generic:Conn_01x05
- U1: footprint Package_DFN_QFN:QFN-16-1EP_3x3mm_P0.5mm_EP1.45x1.45mm -> (none)
Connections:
- net labels removed: BB_IOUT
- wire segments 154 -> 165
Other:
- note added: "I2C: ADD=GND, 0x69\n ADD=Vcc, 0x6F"
- note removed: "Gain = 20V/V\nBB_IOUT = Iout x 2.0\n1.5A = 3.0V"
- moved on the sheet: C5, C9, R1, R2

Commit message: More work on board layouts
Parts:
- added MTH5: Mount Hole, Rays Footprints:Mount-Hole-#6, symbol Connector_Generic:Conn_01x01
- added TP4, TP5: 0.1\" Header, Connector_PinHeader_2.54mm:PinHeader_1x02_P2.54mm_Vertical, symbol Connector_Generic:Conn_01x02
- added TP6: Output Power, Connector_PinHeader_2.54mm:PinHeader_1x02_P2.54mm_Vertical, symbol Connector_Generic:Conn_01x02
- added TP7: Power Debug, Connector_PinHeader_2.54mm:PinHeader_1x02_P2.54mm_Vertical, symbol Connector_Generic:Conn_01x02
- TP2: value Output Power -> GND Debug; footprint Connector_PinHeader_2.54mm:PinHeader_1x06_P2.54mm_Vertical -> Connector_PinHeader_2.54mm:PinHeader_1x02_P2.54mm_Vertical; symbol Connector_Generic:Conn_01x06 -> Connector_Generic:Conn_01x02
- TP3: footprint Connector_PinHeader_2.54mm:PinHeader_1x05_P2.54mm_Vertical -> Connector_JST:JST_XH_B5B-XH-A_1x05_P2.50mm_Vertical
- U1: footprint (none) -> Rays Footprints:MP8862GQ
- gave numbers to parts that had none: 1
Connections:
- net +5V: now also TP5.1 (Pin_1), TP5.2 (Pin_2)
- net GND: now also TP2.2 (Pin_2), TP4.1 (Pin_1), TP4.2 (Pin_2), TP6.1 (Pin_1), TP6.2 (Pin_2); no longer TP2.4 (Pin_4), TP2.5 (Pin_5), TP2.6 (Pin_6)
- net SCL: now also TP3.3 (Pin_3); no longer TP3.4 (Pin_4)
- net SDA: now also TP3.4 (Pin_4); no longer TP3.3 (Pin_3)
- net VOUT: now also TP7.1 (Pin_1), TP7.2 (Pin_2); no longer TP2.2 (Pin_2), TP2.3 (Pin_3)
- net at R5.1, R7.2: now also U2.10 (Vin+); no longer U2.9 (Vin-)
- net at C7.2, C8.1, R5.2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: now also U2.9 (Vin-); no longer U2.10 (Vin+)
Changed lines of the file:
@@
 	7400 2800 7400 2750
 $Comp
-L Connector_Generic:Conn_01x06 TP2
+L Connector_Generic:Conn_01x02 TP2
 U 1 1 5F38C3AA
 P 9150 2500
-F 0 "TP2" H 9100 2950 50  0000 L CNN
-F 1 "Output Power" H 8900 2850 50  0000 L CNN
-F 2 "Connector_PinHeader_2.54mm:PinHeader_1x06_P2.54mm_Vertical" H 9350 2500 50  0001 C CNN
+F 0 "TP2" H 9300 2250 50  0000 L CNN
+F 1 "GND Debug" H 9250 2150 50  0000 L CNN
+F 2 "Connector_PinHeader_2.54mm:PinHeader_1x02_P2.54mm_Vertical" H 9350 2500 50  0001 C CNN
 F 3 "" H 9350 2500 50  0001 C CNN
 	1    9150 2500
@@
 F 0 "TP3" H 2808 4870 50  0000 L CNN
 F 1 "Mount Hole" H 2808 4779 50  0000 L CNN
-F 2 "Connector_PinHeader_2.54mm:PinHeader_1x05_P2.54mm_Vertical" H 2950 4750 50  0001 C CNN
+F 2 "Connector_JST:JST_XH_B5B-XH-A_1x05_P2.50mm_Vertical" H 2950 4750 50  0001 C CNN
 F 3 "" H 2950 4750 50  0001 C CNN
 	1    2750 4750
@@
 	2000 2850 2000 2800
 Connection ~ 2000 2800
-Wire Wire Line
-	8950 2400 8900 2400
-Wire Wire Line
-	8900 2400 8900 2500
 Connection ~ 8900 2500
 Wire Wire Line
 	8900 2500 8950 2500
 Wire Wire Line
-	8900 2400 8900 2300
-Wire Wire Line
-	8900 2300 8950 2300
-Connection ~ 8900 2400
-Wire Wire Line
 	8950 2600 8900 2600
-Wire Wire Line
-	8900 2600 8900 2700
-Wire Wire Line
-	8900 2700 8950 2700
 $Comp
 L power:GND #PWR0113
 U 1 1 5F669595
-P 8850 2700
-F 0 "#PWR0113" H 8850 2450 50  0001 C CNN
-F 1 "GND" H 8855 2527 50  0001 C CNN
-F 2 "" H 8850 2700 50  0001 C CNN
-F 3 "" H 8850 2700 50  0001 C CNN
-	1    8850 2700
+P 8850 3000
+F 0 "#PWR0113" H 8850 2750 50  0001 C CNN
+F 1 "GND" H 8855 2827 50  0001 C CNN
+F 2 "" H 8850 3000 50  0001 C CNN
+F 3 "" H 8850 3000 50  0001 C CNN
+	1    8850 3000
 	0    1    1    0
 $EndComp
-Wire Wire Line
-	8850 2700 8900 2700
-Connection ~ 8900 2700
-Wire Wire Line
-	8900 2800 8950 2800
-Wire Wire Line
-	8900 2700 8900 2800
 Wire Wire Line
 	4700 2500 5500 2500
@@
 $EndComp
 Wire Wire Line
-	8900 2300 8900 2100
-Connection ~ 8900 2300
-Wire Wire Line
 	7750 2500 7750 2450
 Connection ~ 7750 2500
@@
 	7600 1450 7650 1450
 Wire Wire Line
-	6800 1550 6750 1550
-Wire Wire Line
-	6350 1450 6350 2500
-Wire Wire Line
-	6750 1550 6750 2500
-Wire Wire Line
-	6350 1450 6800 1450
-Wire Wire Line
 	8850 2100 8900 2100
 Wire Wire Line
@@
 Text GLabel 2450 4650 0    50   Input ~ 0
 BB_ALERT
+Text GLabel 2450 4850 0    50   Input ~ 0
+SDA
 Text GLabel 2450 4750 0    50   Input ~ 0
-SDA
-Text GLabel 2450 4850 0    50   Input ~ 0
 SCL
 $Comp
@@
 F 0 "U1" H 4250 4915 50  0000 C CNN
 F 1 "MP8862GQ" H 4250 4824 50  0000 C CNN
-F 2 "" H 4050 3400 50  0001 C CNN
+F 2 "Rays Footprints:MP8862GQ" H 4050 3400 50  0001 C CNN
 F 3 "" H 4050 3400 50  0001 C CNN
 	1    4050 3400
@@
 $EndComp
 $Comp
-L Device:R_US R?
+L Device:R_US R6
 U 1 1 5EEDD165
 P 3500 3300
-F 0 "R?" V 3500 2950 50  0000 C CNN
+F 0 "R6" V 3500 2950 50  0000 C CNN
 F 1 "DNP" V 3600 2950 50  0000 C CNN
 F 2 "Rays Footprints:R_0805_HandSoldering" V 3540 3290 50  0001 C CNN
@@
 	3700 3300 3700 3150
 $Comp
-L power:GND #PWR?
+L power:GND #PWR0119
 U 1 1 5EEED5A8
 P 3300 3350
-F 0 "#PWR?" H 3300 3100 50  0001 C CNN
+F 0 "#PWR0119" H 3300 3100 50  0001 C CNN
 F 1 "GND" H 3305 3177 50  0001 C CNN
 F 2 "" H 3300 3350 50  0001 C CNN
@@
 Text Notes 1700 3400 0    79   ~ 0
 I2C: ADD=GND, 0x69\n     ADD=Vcc, 0x6F
+Wire Wire Line
+	6750 1450 6800 1450
+Wire Wire Line
+	6750 1450 6750 2500
+Wire Wire Line
+	6800 1550 6350 1550
+Wire Wire Line
+	6350 1550 6350 2500
+$Comp
+L Connector_Generic:Conn_01x02 TP4
+U 1 1 5EF388A9
+P 4200 4900
+F 0 "TP4" V 4400 4800 50  0000 L CNN
+F 1 "0.1\" Header" V 4300 4650 50  0000 L CNN
+F 2 "Connector_PinHeader_2.54mm:PinHeader_1x02_P2.54mm_Vertical" H 4400 4900 50  0001 C CNN
+F 3 "" H 4400 4900 50  0001 C CNN
+	1    4200 4900
+	0    -1   -1   0
+$EndComp
+$Comp
+L power:GND #PWR0120
+U 1 1 5EF39664
+P 4250 5200
+F 0 "#PWR0120" H 4250 4950 50  0001 C CNN
+F 1 "GND" H 4255 5027 50  0001 C CNN
+F 2 "" H 4250 5200 50  0001 C CNN
+F 3 "" H 4250 5200 50  0001 C CNN
+	1    4250 5200
+	1    0    0    -1
+$EndComp
+Wire Wire Line
+	4200 5100 4200 5150
+Wire Wire Line
+	4200 5150 4250 5150
+Wire Wire Line
+	4300 5150 4300 5100
+Wire Wire Line
+	4250 5200 4250 5150
+Connection ~ 4250 5150
+Wire Wire Line
+	4250 5150 4300 5150
+$Comp
+L Connector_Generic:Conn_01x02 TP5
+U 1 1 5EF5081B
+P 3950 5250
+F 0 "TP5" V 3300 5150 50  0000 L CNN
+F 1 "0.1\" Header" V 3400 4950 50  0000 L CNN
+F 2 "Connector_PinHeader_2.54mm:PinHeader_1x02_P2.54mm_Vertical" H 4150 5250 50  0001 C CNN
+F 3 "" H 4150 5250 50  0001 C CNN
+	1    3950 5250
+	0    1    1    0
+$EndComp
+Wire Wire Line
+	3950 5050 3950 5000
+Wire Wire Line
+	3950 5000 3900 5000
+Wire Wire Line
+	3850 5000 3850 5050
+Connection ~ 3900 5000
+Wire Wire Line
+	3900 5000 3850 5000
+Text GLabel 3850 4900 0    50   Input ~ 0
++5V
+Wire Wire Line
+	3850 4900 3900 4900
+Wire Wire Line
+	3900 4900 3900 5000
+$Comp
+L Connector_Generic:Conn_01x01 MTH5
+U 1 1 5EF6BD72
+P 5200 6400
+F 0 "MTH5" H 5258 6520 50  0000 L CNN
+F 1 "Mount Hole" H 5258 6429 50  0000 L CNN
+F 2 "Rays Footprints:Mount-Hole-#6" H 5400 6400 50  0001 C CNN
+F 3 "~" H 5400 6400 50  0001 C CNN
+	1    5200 6400
+	1    0    0    -1
+$EndComp
+$Comp
+L Connector_Generic:Conn_01x02 TP6
+U 1 1 5EF75978
+P 9150 2750
+F 0 "TP6" H 9300 3000 50  0000 L CNN
+F 1 "Output Power" H 9250 2900 50  0000 L CNN
+F 2 "Connector_PinHeader_2.54mm:PinHeader_1x02_P2.54mm_Vertical" H 9350 2750 50  0001 C CNN
+F 3 "" H 9350 2750 50  0001 C CNN
+	1    9150 2750
+	1    0    0    -1
+$EndComp
+Wire Wire Line
+	8950 2250 8900 2250
+Connection ~ 8900 2250
+Wire Wire Line
+	8900 2250 8900 2100
+Wire Wire Line
+	8950 2350 8900 2350
+Connection ~ 8900 2350
+Wire Wire Line
+	8900 2250 8900 2350
+Wire Wire Line
+	8900 2850 8950 2850
+Wire Wire Line
+	8950 2750 8900 2750
+Connection ~ 8900 2750
+Wire Wire Line
+	8900 2750 8900 2850
+$Comp
+L Connector_Generic:Conn_01x02 TP7
+U 1 1 5EF9890A
+P 9150 2250
+F 0 "TP7" H 9300 2250 50  0000 L CNN
+F 1 "Power Debug" H 9250 2150 50  0000 L CNN
+F 2 "Connector_PinHeader_2.54mm:PinHeader_1x02_P2.54mm_Vertical" H 9350 2250 50  0001 C CNN
+F 3 "" H 9350 2250 50  0001 C CNN
+	1    9150 2250
+	1    0    0    -1
+$EndComp
+Wire Wire Line
+	8900 2350 8900 2500
+Wire Wire Line
+	8850 3000 8900 3000
+Wire Wire Line
+	8900 3000 8900 2850
+Connection ~ 8900 2850
+Wire Wire Line
+	8900 2600 8900 2750
 $EndSCHEMATC
