File: lab-supply-usb-buck-boost.kicad_pcb (KiCad board)
At the start: 2 copper layers, 94 x 66 mm, 49 parts, among them Q1 Q_NPN_BCE, U1 MP8862GQ, U2 INA220, U3 MAX1719EUT

Commit message: Lots of updates
Parts:
- moved TP3 30.0 mm to (153.3, 114.3), turned to 180 degrees
- moved TP6 14.2 mm to (163.2, 92.8)
- moved TP7 13.5 mm to (163.2, 79.9)
Routing:
- net +5V: track 236.9 -> 203.1 mm, vias 3 -> 0
- net VOUT: track 71.2 -> 62.4 mm
- net SDA: track 148.6 -> 156.2 mm, vias 4 -> 7
- net SCL: track 153.6 -> 161.1 mm, vias 3 -> 6
- net BB_ALERT: track 88.3 -> 81.0 mm
