File: lab-supply-control-board.kicad_pcb (KiCad board)
At the start: 2 copper layers, 94 x 66 mm, 88 parts, among them J1 JST, J10 USB-Micro, J11 0.1" Header, J12 1x05 JST, J13 1x04 JST, J14 0.1" Header, J15 0.1" Header, J2 JST, J3 JST, J4 0.1" Header, J5 0.1" Header, J6 AVR-ISP-6, J7 0.1" Header, J8 0.1" Header, J9 0.1" Header, Q3 2N3904, Q4 2N3904, Q5 2N3904, Q7 BSS138, U1 MCP4716A0T-ECH, U2 ATmega328P-AU, U4 LM4040DBZ-2.5, U5 MCP4716A1T-ECH, U7 FT232RL, U8 MCP6002-xSN, Y1 Crystal_GND24

Commit message: finalized before PCB orders
Parts:
- removed Q7: BSS138, Package_TO_SOT_SMD:SOT-23
- removed R36, R37: 10k, Rays Footprints:R_0805_HandSoldering
- moved J5 42.2 mm to (78.9, 107.1), turned to 90 degrees
- moved D6 32.0 mm to (109.1, 116.4), turned to 180 degrees
- moved R48 31.9 mm to (109.1, 113.8), turned to 180 degrees
- moved J9 27.2 mm to (100.3, 115.4), turned to 90 degrees
- moved R44 15.5 mm to (117.8, 101.3), turned to 90 degrees
- moved R32 12.7 mm to (120.3, 101.3)
- moved R38 12.7 mm to (120.3, 106.8)
- moved R43 12.4 mm to (117.8, 106.8), turned to 270 degrees
- moved R30 10.8 mm to (115.3, 101.3)
- moved J10 10.2 mm to (75.1, 76.2)
- moved C11 10.2 mm to (84.3, 68.5)
- moved R26 10.2 mm to (105.1, 106.9)
- moved R27 10.2 mm to (105.1, 101.3)
- moved D3 8.57 mm to (84.3, 86.6)
- moved D4 8.57 mm to (86.7, 86.6)
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Connections:
- J12 pad 1: (no net) -> BB_ALERT
- J5 pad 1: GND -> Net-(J5-Pad1)
- J5 pad 2: DISP_RESET_3.3 -> DISP_DC_3.3
- J5 pad 3: Net-(J5-Pad3) -> DISP_RESET_3.3
- J5 pad 4: SCK_3.3 -> DISP_CS_3.3
- J5 pad 7: DISP_DC_3.3 -> SCK_3.3
- J5 pad 8: DISP_CS_3.3 -> GND
- R15 pad 2: Net-(J5-Pad3) -> Net-(J5-Pad1)
- R18 pad 2: Net-(J5-Pad3) -> Net-(J5-Pad1)
- R22 pad 2: Net-(J5-Pad3) -> Net-(J5-Pad1)
Routing:
- net Net-(J5-Pad1): track 0.00 -> 57.6 mm
- net +3.3V: track 90.0 -> 41.3 mm, vias 4 -> 3
- net DISP_DC_3.3: track 16.9 -> 54.1 mm
- net DISP_RESET_3.3: track 26.1 -> 59.8 mm
- net DISP_CS_3.3: track 16.9 -> 47.7 mm
- net MOSI_3.3: track 16.9 -> 47.2 mm
- net MISO_3.3: track 16.9 -> 45.6 mm
- net SCK_3.3: track 16.9 -> 45.3 mm
- net DISP_RESET: track 41.5 -> 14.2 mm
- net +5V: track 451.2 -> 469.4 mm, vias 4 -> 5
- net Net-(J5-Pad3): track 15.9 -> 0.00 mm
- net DISP_DC: track 38.5 -> 50.5 mm, vias 2 -> 3
- net USB_D-: track 17.3 -> 28.6 mm, vias 2 -> 4
- net USB_D+: track 16.0 -> 26.8 mm
- net SCK: track 84.8 -> 94.4 mm
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Other:
- net class Default: clearance 0.2032 -> 0.1778
- rule trace_clearance: 0.2032 -> 0.1778
- board text added: "Buttons"
- board text added: "Display"
- board text removed: "2.16"
- board text removed: "DISPLAY"
