File: lab-supply-usb-boost-buck.sch (KiCad schematic (older format))
At the start: 69 parts, among them Q1 Q_NPN_BCE, U1 INA220, U2 MAX17572, U3 MAX1719EUT, U4 MAX17250, U5 MCP4716AxT-ECH, U6 INA220, U7 LM4040DBZ-2.5, U8 MCP4716AxT-ECH

Commit message: finalized before PCB orders
Parts:
- added R16, R17: DNP, Rays Footprints:R_0805_HandSoldering, symbol Device:R_US
- added R4: 1k, Rays Footprints:R_0805_HandSoldering, symbol Device:R_US
- added TP11, TP12, TP13: 0.1\" Header, Connector_PinHeader_2.54mm:PinHeader_1x01_P2.54mm_Vertical, symbol Connector_Generic:Conn_01x01
- C1: value 10u -> 10u/35V
- C10: value 5.6n -> 10n
- C14: value 10u -> 10u/25V
- C15: value 10n -> 4.7n
- C7: value 10u -> 100u/25V; footprint Rays Footprints:C_1210_HandSoldering -> Capacitor_SMD:CP_Elec_6.3x5.9
- L1: value 2.2uH -> 15uH
- L2: value 15uH -> 2.2uH
- R12: value 0 -> 84.5k
- R15: value 0 -> 10k
Connections:
- net 2.5V_REF: now also TP13.1 (Pin_1)
- net DAC_BOOST: now also TP12.1 (Pin_1)
- net DAC_BUCK: now also TP11.1 (Pin_1)
- net GND: now also R17.1; no longer U3.5 (~SHDN)
- net VIN_BUCK: now also U6.8 (Vbus); no longer U2.2 (EN/UVLO)
- net at C11.1, R7.1, U3.2 (IN): now also U3.5 (~SHDN)
- net VL: now reaches C19.2, U4.1 (VL)
- net VL: now also R16.1
- net at C16.2, C17.2, U4.10 (PVH)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: now also C15.2; no longer C15.1
- net at U4.5 (ISET): now also R16.2, R17.2
- net at U4.8 (OUT): now also C14.2, R11.2, TP8.1 (Pin_1), U6.10 (Vin+), R4.2
- net ENABLE: now reaches TP3.2 (Pin_2)
- net ENABLE: now also U2.2 (EN/UVLO)
- new net: C9.2, L2.2, U4.11 (LX), U4.12 (LX)
- new net: C15.1, R12.2, R4.1
Other:
- note added: "0V-15Vin @1A"
- note added: "Open: Ipk=1.85A\nAGND: Ipk=2.7A\nVL: Ipk = 3.5A"
- note added: "XAL4020-222ME"
- note added: "XAL4040-153ME"
- note removed: "0V-0.9Vin @1.5A"
- moved on the sheet: C11, C12, C13, C14, C15, C18, C20, C21, C22, C5, JP3, JP4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
